Commit message: config xacro

File: src/skt_description/robot/visual/castor.xacro (robot description, xacro)
@@ -38,9 +38,9 @@
   <xacro:macro name="castor_set_graphics" params="">
     <xacro:castor_graphics
-      name="left_front"
+      name="front"
       translation_x="${CASTOR_SEPARATION_X/2}"
       translation_y="${CASTOR_SEPARATION_Y/2}"
     />
-    <xacro:castor_graphics
+    <!-- <xacro:castor_graphics
       name="right_front"
       translation_x="${CASTOR_SEPARATION_X/2}"
@@ -56,5 +56,5 @@
       translation_x="${-CASTOR_SEPARATION_X/2}"
       translation_y="${-CASTOR_SEPARATION_Y/2}"
-    />
+    /> -->
   </xacro:macro>
 </robot>

File: src/skt_description/robot/visual/sensor.xacro (robot description, xacro)
@@ -7,5 +7,5 @@
       <parent link="base_link" />
       <child link="imu_link" />
-      <origin xyz="0 0 0" rpy="0 0 0" />
+      <origin xyz="0 0 0" rpy="0 -0.169 0" />
     </joint>
   </xacro:macro>

File: src/skt_description/robot/visual/skt_rviz.xacro (robot description, xacro)
@@ -11,4 +11,7 @@
         <xacro:include filename="${visual_path}/castor.xacro"/>
         <xacro:castor_set_graphics/>
+        <!-- Add wheels -->
+        <xacro:include filename="${visual_path}/wheel.xacro"/>
+        <xacro:wheel_set_graphics/>
         <!-- Add sensor link -->
         <xacro:include filename="${visual_path}/sensor.xacro"/>
