Commit message: check point

File: src/skt_description/robot/visual/sensor.xacro (robot description, xacro)
@@ -7,5 +7,5 @@
       <parent link="base_link" />
       <child link="imu_link" />
-      <origin xyz="0 0 0" rpy="0 -0.169 0" />
+      <origin xyz="0 0 0" rpy="0 0 0" />
     </joint>
   </xacro:macro>
